Commit message: urdf correction

File: ros2/src/mfr/config/sim_car.urdf (robot description, URDF)
Before this commit: robot sim_car, 3 links, 2 joints
Links:
- removed link fsd/FSCar
- added link fsds/FSCar
Joints:
- removed joint base_joint
- removed joint base_to_FSC
- added joint FSDS_to_base_footprint: type fixed, parent fsds/FSCar, child base_link, origin xyz=0 0 0 rpy=0 0 0
- added joint footprint_link: type fixed, parent base_link, child base_footprint, origin xyz=0 0 0 rpy=0 0 0

Commit message: correction on urdf and lidar positioning

File: ros2/src/mfr/config/sim_car.urdf (robot description, URDF)
Before this commit: robot sim_car, 3 links, 2 joints
Joints:
- joint FSDS_to_base_footprint: child base_link -> base_footprint
- joint footprint_link: child base_footprint -> base_link; origin xyz=0 0 0 rpy=0 0 0 -> xyz=0 0 0.20 rpy=0 0 0; parent base_link -> base_footprint
